Commit message: init

File: src/erc_gazebo_sensors/urdf/erc_bot.urdf (robot description, URDF)
Before this commit: robot erc_bot, 9 links, 8 joints
Links:
- removed link camera_link
- removed link camera_link_optical
- removed link scan_link
- link base_link: geometry collision box size=.4 .2 .1; visual box size=.4 .2 .1
- link front_left_wheel: geometry collision cylinder length=.05 radius=.1; visual cylinder length=.05 radius=.1
- link front_right_wheel: geometry collision cylinder length=.05 radius=.1; visual cylinder length=.05 radius=.1
- link rear_left_wheel: geometry collision cylinder length=.05 radius=.1; visual cylinder length=.05 radius=.1
- link rear_right_wheel: geometry collision cylinder length=.05 radius=.1; visual cylinder length=.05 radius=.1
Joints:
- removed joint camera_joint
- removed joint camera_optical_joint
- removed joint scan_joint

Commit message: Complete Session 4: Perception and YOLOv8 Object Hunt

File: src/erc_gazebo_sensors/urdf/erc_bot.urdf (robot description, URDF)
Before this commit: robot erc_bot, 5 links, 4 joints
Links:
- removed link front_caster_wheel
- added link camera_link, mass 0.1; collision box size=.03 .03 .03; visual box size=.03 .03 .03
- added link camera_link_optical
- added link front_left_wheel, mass 5.0; collision cylinder length=.05 radius=.1; visual cylinder length=.05 radius=.1
- added link front_right_wheel, mass 5.0; collision cylinder length=.05 radius=.1; visual cylinder length=.05 radius=.1
- added link imu_link
- added link scan_link, mass 1e-5; collision box size=.06 .06 .06; visual box size=.06 .06 .06
Joints:
- removed joint front_caster_wheel_joint
- added joint camera_joint: type fixed, parent base_link, child camera_link, origin xyz=0.225 0 0.075 rpy=0 0 0, axis 0 1 0
- added joint camera_optical_joint: type fixed, parent camera_link, child camera_link_optical, origin xyz=0 0 0 rpy=-1.5707 0 -1.5707
- added joint front_left_wheel_joint: type continuous, parent base_link, child front_left_wheel, origin xyz=0.15 0.15 0 rpy=0 0 0, axis 0 1 0, limit effort=100 velocity=10
- added joint front_right_wheel_joint: type continuous, parent base_link, child front_right_wheel, origin xyz=0.15 -0.15 0 rpy=0 0 0, axis 0 1 0, limit effort=100 velocity=10
- added joint imu_joint: type fixed, parent base_link, child imu_link, origin xyz=0 0 0 rpy=0 0 0
- added joint scan_joint: type fixed, parent base_link, child scan_link, origin xyz=0.0 0 0.15 rpy=0 0 0, axis 0 1 0
